File: FBF_STM32CoreBoard.sch (KiCad schematic (older format))
At the start: 40 parts, among them J1 SWD_STM32, J2 DB9, P1 CONN_02X03, SW1 SW_PUSH, U1 NCP1117ST33T3G, U2 STM32F103RT6, U3 SP3232E, Y1 327680HZ, Y2 8MHZ/5032

Commit message: trying to finish the project
Parts:
- added P? (x4): CONN_01X12, symbol CONN_01X12
Connections:
- net KEY0 is gone; now on net PC13: SW?.2
- net +3V3: now also P?.4 (P4)
- net +5V: now also P?.1 (P1)
- net GND: now also P?.1 (P1), P?.2 (P2), P?.3 (P3)
- net NRST: now also P?.3 (P3)
- net PA0: now also P?.7 (P7)
- net PA1: now also P?.6 (P6)
- net PA11: now also P?.3 (P3)
- net PA12: now also P?.2 (P2)
- net PA15: now also P?.1 (P1)
- net PA2: now also P?.5 (P5)
- net PA3: now also P?.12 (P12)
- net PA4: now also P?.11 (P11)
- net PA5: now also P?.10 (P10)
- net PA6: now also P?.9 (P9)
- net PA7: now also P?.8 (P8)
- net PA8: now also P?.4 (P4)
- net PB0: now also P?.5 (P5)
- net PB1: now also P?.4 (P4)
- net PB10: now also P?.3 (P3)
- net PB11: now also P?.2 (P2)
- net PB12: now also P?.12 (P12)
- net PB13: now also P?.11 (P11)
- net PB14: now also P?.10 (P10)
- net PB15: now also P?.9 (P9)
- net PB3: now also P?.8 (P8)
- net PB4: now also P?.7 (P7)
- net PB5: now also P?.6 (P6)
- net PB6: now also P?.5 (P5)
- net PB7: now also P?.4 (P4)
- net PB8: now also P?.2 (P2)
- net PB9: now also P?.1 (P1)
- net PC0: now also P?.11 (P11)
- net PC1: now also P?.10 (P10)
- net PC10: now also P?.12 (P12)
- net PC11: now also P?.11 (P11)
- net PC12: now also P?.10 (P10)
- net PC2: now also P?.9 (P9)
- net PC3: now also P?.8 (P8)
- net PC4: now also P?.7 (P7)
- net PC5: now also P?.6 (P6)
- net PC6: now also P?.8 (P8)
- net PC7: now also P?.7 (P7)
- net PC8: now also P?.6 (P6)
- net PC9: now also P?.5 (P5)
- net PD2: now also P?.9 (P9)
- no-connect marks 0 -> 1
Other:
- moved on the sheet: C1, C2, P1, R5, R6, U1

Commit message: check the schematic and modify some connection
Parts:
- added C?: 10uF/Tantalum, symbol C
- added R?: 10K/1%/0603, symbol R
- C2: value 22uF/Tantalum -> 100nF/5%/0603
- C7: value 10uF/10%/6032/Tantalum -> 1UF/Tantalum
- R2: value R -> 0
Connections:
- net KEY1 is gone; now on net PC0: SW?.2
- net +3V3: now also C?.2, R?.2
- net GND: now also C?.1
- net NRST2: now also R?.1
- net PA8: now also D3.1 (K)
- net PD2: now also D2.1 (K)
- removed net LED_SHOW_RUN: D2.1 (K), D3.1 (K)
Other:
- moved on the sheet: D1, R1, R2
Changed lines of the file:
@@
 P 3050 5000
 F 0 "C7" V 3000 4850 50  0000 L CNN
-F 1 "10uF/10%/6032/Tantalum" H 2600 4750 50  0000 L CNN
+F 1 "1UF/Tantalum" H 2750 4800 50  0000 L CNN
 F 2 "" H 3088 4850 50  0000 C CNN
 F 3 "" H 3050 5000 50  0000 C CNN
@@
 L R R2
 U 1 1 57E6C0E0
-P 3000 4100
-F 0 "R2" V 3080 4100 50  0000 C CNN
-F 1 "R" V 3000 4100 50  0000 C CNN
-F 2 "" V 2930 4100 50  0000 C CNN
-F 3 "" H 3000 4100 50  0000 C CNN
-	1    3000 4100
+P 2950 4100
+F 0 "R2" V 3030 4100 50  0000 C CNN
+F 1 "0" V 2950 4100 50  0000 C CNN
+F 2 "" V 2880 4100 50  0000 C CNN
+F 3 "" H 2950 4100 50  0000 C CNN
+	1    2950 4100
 	0    1    1    0
 $EndComp
@@
 Connection ~ 3550 3750
 Wire Wire Line
-	2850 4100 2500 4100
+	2800 4100 2500 4100
 Text Label 2500 4100 0    60   ~ 0
 NRST
@@
 L R R1
 U 1 1 57E74247
-P 2850 4550
-F 0 "R1" V 2930 4550 50  0000 C CNN
-F 1 "10k/1%/0603" V 2750 4450 50  0000 C CNN
-F 2 "" V 2780 4550 50  0000 C CNN
-F 3 "" H 2850 4550 50  0000 C CNN
-	1    2850 4550
+P 1450 5900
+F 0 "R1" V 1530 5900 50  0000 C CNN
+F 1 "10k/1%/0603" V 1350 5800 50  0000 C CNN
+F 2 "" V 1380 5900 50  0000 C CNN
+F 3 "" H 1450 5900 50  0000 C CNN
+	1    1450 5900
 	0    1    1    0
 $EndComp
@@
 L +3V3 #PWR017
 U 1 1 57E74375
-P 2550 4550
-F 0 "#PWR017" H 2550 4400 50  0001 C CNN
-F 1 "+3V3" H 2550 4690 50  0000 C CNN
-F 2 "" H 2550 4550 50  0000 C CNN
-F 3 "" H 2550 4550 50  0000 C CNN
-	1    2550 4550
+P 1150 5900
+F 0 "#PWR017" H 1150 5750 50  0001 C CNN
+F 1 "+3V3" H 1150 6040 50  0000 C CNN
+F 2 "" H 1150 5900 50  0000 C CNN
+F 3 "" H 1150 5900 50  0000 C CNN
+	1    1150 5900
 	0    -1   -1   0
 $EndComp
 Wire Wire Line
-	2550 4550 2700 4550
+	1150 5900 1300 5900
 $Comp
 L LED D1
 U 1 1 57E744B4
-P 3350 4550
-F 0 "D1" H 3350 4650 50  0000 C CNN
-F 1 "LED_RED_Power" H 3350 4450 50  0000 C CNN
-F 2 "" H 3350 4550 50  0000 C CNN
-F 3 "" H 3350 4550 50  0000 C CNN
-	1    3350 4550
+P 1950 5900
+F 0 "D1" H 1950 6000 50  0000 C CNN
+F 1 "LED_RED_Power" H 1950 5800 50  0000 C CNN
+F 2 "" H 1950 5900 50  0000 C CNN
+F 3 "" H 1950 5900 50  0000 C CNN
+	1    1950 5900
 	-1   0    0    1
 $EndComp
 Wire Wire Line
-	3000 4550 3150 4550
+	1600 5900 1750 5900
 $Comp
 L GND #PWR018
 U 1 1 57E7460F
-P 3650 4550
-F 0 "#PWR018" H 3650 4300 50  0001 C CNN
-F 1 "GND" H 3650 4400 50  0000 C CNN
-F 2 "" H 3650 4550 50  0000 C CNN
-F 3 "" H 3650 4550 50  0000 C CNN
-	1    3650 4550
+P 2250 5900
+F 0 "#PWR018" H 2250 5650 50  0001 C CNN
+F 1 "GND" H 2250 5750 50  0000 C CNN
+F 2 "" H 2250 5900 50  0000 C CNN
+F 3 "" H 2250 5900 50  0000 C CNN
+	1    2250 5900
 	0    -1   -1   0
 $EndComp
 Wire Wire Line
-	3550 4550 3650 4550
-Text Label 3050 4550 0    60   ~ 0
+	2150 5900 2250 5900
+Text Label 1650 5900 0    60   ~ 0
 POWER_LED
 $Comp
@@
 	8450 3900 8600 3900
 Text Label 8600 3900 0    60   ~ 0
-LED_SHOW_RUN
+PA8
 $Comp
 L NCP1117ST33T3G U1
@@
 L +3V3 #PWR022
 U 1 1 57E7EF0E
-P 2000 4600
-F 0 "#PWR022" H 2000 4450 50  0001 C CNN
-F 1 "+3V3" H 2000 4740 50  0000 C CNN
-F 2 "" H 2000 4600 50  0000 C CNN
-F 3 "" H 2000 4600 50  0000 C CNN
-	1    2000 4600
-	0    1    1    0
-$EndComp
-Wire Wire Line
-	1850 4600 2000 4600
+P 2050 4450
+F 0 "#PWR022" H 2050 4300 50  0001 C CNN
+F 1 "+3V3" H 2050 4590 50  0000 C CNN
+F 2 "" H 2050 4450 50  0000 C CNN
+F 3 "" H 2050 4450 50  0000 C CNN
+	1    2050 4450
+	1    0    0    -1
+$EndComp
+Wire Wire Line
+	1850 4600 2350 4600
 $Comp
 L C C2
@@
 P 1900 4800
 F 0 "C2" V 1850 4650 50  0000 L CNN
-F 1 "22uF/Tantalum" H 1650 5100 50  0000 L CNN
+F 1 "100nF/5%/0603" H 1650 5100 50  0000 L CNN
 F 2 "" H 1938 4650 50  0000 C CNN
 F 3 "" H 1900 4800 50  0000 C CNN
@@
 Connection ~ 1900 4600
 Wire Wire Line
-	1000 4950 1900 4950
+	1000 4950 2350 4950
 Connection ~ 1450 4950
 $Comp
@@
 	8450 3600 8600 3600
 Text Label 8600 3600 0    60   ~ 0
-LED_SHOW_RUN
+PD2
 Wire Wire Line
 	4600 3300 4450 3300
@@
 PC13
 Text Label 5650 5400 1    60   ~ 0
-KEY1
+PC0
 Text Label 5950 5400 1    60   ~ 0
 KEY2
@@
 	4750 5800 4850 5800
 NoConn ~ 1400 2900
+$Comp
+L R R?
+U 1 1 57ECA20E
+P 2950 3900
+F 0 "R?" V 3030 3900 50  0000 C CNN
+F 1 "10K/1%/0603" V 2900 3850 50  0000 C CNN
+F 2 "" V 2880 3900 50  0000 C CNN
+F 3 "" H 2950 3900 50  0000 C CNN
+	1    2950 3900
+	0    1    1    0
+$EndComp
+Wire Wire Line
+	3150 4100 3100 4100
+Wire Wire Line
+	3100 3900 3150 3900
+Connection ~ 3150 3900
+Wire Wire Line
+	2500 3900 2800 3900
+$Comp
+L +3V3 #PWR?
+U 1 1 57ECA90B
+P 2500 3900
+F 0 "#PWR?" H 2500 3750 50  0001 C CNN
+F 1 "+3V3" H 2500 4040 50  0000 C CNN
+F 2 "" H 2500 3900 50  0000 C CNN
+F 3 "" H 2500 3900 50  0000 C CNN
+	1    2500 3900
+	0    -1   -1   0
+$EndComp
+$Comp
+L C C?
+U 1 1 57ECECC1
+P 2350 4800
+F 0 "C?" V 2300 4650 50  0000 L CNN
+F 1 "10uF/Tantalum" V 2150 4450 50  0000 L CNN
+F 2 "" H 2388 4650 50  0000 C CNN
+F 3 "" H 2350 4800 50  0000 C CNN
+	1    2350 4800
+	-1   0    0    1
+$EndComp
+Wire Wire Line
+	2350 4600 2350 4650
+Wire Wire Line
+	2050 4450 2050 4600
+Connection ~ 2050 4600
+Connection ~ 1900 4950
 $EndSCHEMATC

Commit message: Check the Designation
Parts:
- C1: footprint (none) -> Capacitors_Tantalum_SMD:TantalC_SizeC_EIA-6032_HandSoldering
- C10, C11, C12, C13, C2, C3, C4, C5, C6, C8, C9, D1, D2, D3, FB1: footprint (none) -> Capacitors_SMD:C_0603_HandSoldering
- C19: renamed from C?; footprint (none) -> Capacitors_Tantalum_SMD:TantalC_SizeC_EIA-6032_HandSoldering
- J2: footprint (none) -> Connect:DB9MD
- R1, R2, R3, R4, R5, R6: footprint (none) -> Resistors_SMD:R_0603_HandSoldering
- R7: renamed from R?; footprint (none) -> Resistors_SMD:R_0603_HandSoldering
- U1: footprint (none) -> TO_SOT_Packages_SMD:SOT-223
- gave numbers to parts that had none: 7
Connections:
- net KEY2 is gone; now on net PA0: SW4.2
- net +3V3: now also SW4.1
- no-connect marks 1 -> 11

Commit message: change the properties of the board
Parts:
- U1: symbol NCP1117ST33T3G -> NCP1117ST33T3G-RESCUE-FBF_STM32CoreBoard
- U2: footprint (none) -> FairySpaceFootprint:LQFP64
Changed lines of the file:
@@
 EESchema Schematic File Version 2
+LIBS:FBF_STM32CoreBoard-rescue
 LIBS:power
 LIBS:device
@@
 F 0 "U2" H 4650 2550 60  0000 C CNN
 F 1 "STM32F103RT6" H 4650 1250 60  0000 C CNN
-F 2 "" H 5600 2800 60  0001 C CNN
+F 2 "FairySpaceFootprint:LQFP64" H 5600 2800 60  0001 C CNN
 F 3 "" H 5600 2800 60  0000 C CNN
 	1    5600 2800
@@
 PA8
 $Comp
-L NCP1117ST33T3G U1
+L NCP1117ST33T3G-RESCUE-FBF_STM32CoreBoard U1
 U 1 1 57E7E7AD
 P 1450 4650
